File: stm32_red_pill_old.kicad_pcb (KiCad board)
At the start: 2 copper layers, 59 x 31 mm, 29 parts, among them J1 USB_B_Micro, J2 Conn_01x18, J3 Conn_01x18, SW1 SW_SPDT, U1 STM32F103C8T6, U2 AMS1117-3.3, Y1 16MHZ

Commit message: Initial commit
Parts:
- moved SW1 53.9 mm to (82.6, 100.0), turned to -90 degrees
- moved R1 43.8 mm to (88.6, 100.9), turned to 0 degrees
- moved R3 19.5 mm to (135.4, 93.5), turned to 0 degrees
- moved D1 14.3 mm to (132.5, 93.5), turned to 180 degrees
- moved C10 6.96 mm to (105.8, 95.2)
- moved Y1 6.96 mm to (103.3, 95.9)
- moved C11 6.96 mm to (105.8, 97.2)
- moved C13 6.12 mm to (126.9, 102.2), turned to 180 degrees
- moved C8 5.94 mm to (103.2, 105.6), turned to -90 degrees
- moved C12 5.26 mm to (121.9, 97.1), turned to -90 degrees
- moved C7 5.16 mm to (101.2, 105.6), turned to -90 degrees
- moved FB1 4.40 mm to (102.2, 103.6), turned to 0 degrees
- moved C6 4.12 mm to (108.1, 98.7)
- moved U2 3.96 mm to (126.9, 96.2), turned to 90 degrees
- moved C1 3.90 mm to (111.3, 95.8)
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Routing:
- net +3.3V: track 74.4 -> 109.5 mm, vias 6 -> 10
- net +3.3VA: track 12.4 -> 29.5 mm, vias 2 -> 4
- net VBUS: track 4.60 -> 13.7 mm, vias 6 -> 4
- net /PC15: track 15.2 -> 24.0 mm, vias 0 -> 2
- net /PB9: track 13.7 -> 19.1 mm
- net /PC14: track 13.4 -> 18.0 mm, vias 0 -> 2
- net /USB_D-: track 21.6 -> 17.6 mm
- net /USB_D+: track 21.3 -> 17.2 mm
- net /PA9: track 17.9 -> 13.9 mm
- net /PA10: track 20.2 -> 16.3 mm
- net /PA4: track 18.3 -> 22.1 mm
- net /PA5: track 16.0 -> 19.8 mm
- net /PA3: track 20.7 -> 24.5 mm
- net /PA6: track 13.8 -> 17.5 mm
- net /PA8: track 15.6 -> 12.0 mm
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