File: stm32_red_pill.kicad_sch (KiCad schematic)
At the start: 29 parts, among them J1 USB_B_Micro, J2 Conn_01x18, J3 Conn_01x18, J4 Conn_01x03, U1 STM32F103C8T6, U2 AMS1117-3.3, Y1 16MHZ

Commit message: lib submodule
Parts:
- C1, C2, C3, C4, C9: LCSC (none) -> C1525; MPN C1525 -> (none)
- C10, C11: LCSC (none) -> C32949; MPN C32949 -> (none)
- C12, C13: LCSC (none) -> C45783; MPN C45783 -> (none)
- C5: LCSC (none) -> C19702; MPN C19702 -> (none)
- C6: LCSC (none) -> C15195; MPN C15195 -> (none)
- C7, C8: LCSC (none) -> C52923; MPN C52923 -> (none)
- D1: LCSC (none) -> C2286; MPN C2286 -> (none)
- FB1: LCSC (none) -> C1002; MPN C1002 -> (none)
- J1: LCSC (none) -> C2894326; MPN C2894326 -> (none)
- R1: LCSC (none) -> C25744; MPN C25744 -> (none)
- R2, R3: LCSC (none) -> C25867; MPN C25867 -> (none)
- U1: LCSC (none) -> C8734; MPN C8734 -> (none)
- U2: LCSC (none) -> C6186; MPN C6186 -> (none)
- Y1: LCSC (none) -> C12668; MPN C12668 -> (none)
Changed lines of the file:
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@@
 			)
 		)
-		(property "MPN" "C1525"
+		(property "LCSC" "C1525"
 			(at 85.09 41.91 0)
 			(effects
@@
 			)
 		)
-		(property "MPN" "C45783"
+		(property "LCSC" "C45783"
 			(at 71.12 163.83 0)
 			(effects
@@
 			)
 		)
-		(property "MPN" "C15195"
+		(property "LCSC" "C15195"
 			(at 134.62 41.91 0)
 			(effects
@@
 			)
 		)
-		(property "MPN" "C6186"
+		(property "LCSC" "C6186"
 			(at 55.88 157.48 0)
 			(effects
@@
 			)
 		)
-		(property "MPN" "C1002"
+		(property "LCSC" "C1002"
 			(at 156.21 36.83 0)
 			(effects
@@
 			)
 		)
-		(property "MPN" "C12668"
+		(property "LCSC" "C12668"
 			(at 53.34 73.66 0)
 			(effects
@@
 			)
 		)
-		(property "MPN" "C1525"
+		(property "LCSC" "C1525"
 			(at 72.39 41.91 0)
 			(effects
@@
 			)
 		)
-		(property "MPN" "C32949"
+		(property "LCSC" "C32949"
 			(at 60.96 86.36 0)
 			(effects
@@
 			)
 		)
-		(property "MPN" "C8734"
+		(property "LCSC" "C8734"
 			(at 102.87 87.63 0)
 			(effects
@@
 			)
 		)
-		(property "MPN" "C1525"
+		(property "LCSC" "C1525"
 			(at 59.69 41.91 0)
 			(effects
@@
 			)
 		)
-		(property "MPN" "C45783"
+		(property "LCSC" "C45783"
 			(at 38.1 163.83 0)
 			(effects
@@
 			)
 		)
-		(property "MPN" "C32949"
+		(property "LCSC" "C32949"
 			(at 44.45 86.36 0)
 			(effects
@@
 			)
 		)
-		(property "MPN" "C52923"
+		(property "LCSC" "C52923"
 			(at 147.32 41.91 0)
 			(effects
@@
 			)
 		)
-		(property "MPN" "C2286"
+		(property "LCSC" "C2286"
 			(at 78.74 157.48 0)
 			(effects
@@
 			)
 		)
-		(property "MPN" "C1525"
+		(property "LCSC" "C1525"
 			(at 34.29 58.42 0)
 			(effects
@@
 			)
 		)
-		(property "MPN" "C1525"
+		(property "LCSC" "C1525"
 			(at 46.99 41.91 0)
 			(effects
@@
 			)
 		)
-		(property "MPN" "C25744"
+		(property "LCSC" "C25744"
 			(at 69.85 59.69 0)
 			(effects
@@
 			)
 		)
-		(property "MPN" "C2894326"
+		(property "LCSC" "C2894326"
 			(at 160.02 85.09 0)
 			(effects
@@
 			)
 		)
-		(property "MPN" "C25867"
+		(property "LCSC" "C25867"
 			(at 86.36 163.83 0)
 			(effects
@@
 			)
 		)
-		(property "MPN" "C19702"
+		(property "LCSC" "C19702"
 			(at 34.29 41.91 0)
 			(effects
@@
 			)
 		)
-		(property "MPN" "C25867"
+		(property "LCSC" "C25867"
 			(at 142.24 77.47 0)
 			(effects
@@
 			)
 		)
-		(property "MPN" "C52923"
+		(property "LCSC" "C52923"
 			(at 165.1 41.91 0)
 			(effects
